Commit message: D1 Phase 2c: ★16-DOF 능동 발목 확장 — trot 보행 성공 + 버징↓ + GEARBOX
12-DOF point-foot → 16-DOF 능동발목(발목4 언락, 허리 fixed 유지):
- URDF: 4개 *_foot_joint fixed→revolute(02leg_ocs2_12dof.urdf 백업).
- config: jointNames 12→16(다리별 hip,thigh,calf,foot), Q/R/initialState
  28차원 재작성(발목 Q=10=자세자유도, R=5000). reference nominal foot=0.
- WBC: torqueLimits perLeg 자동(3→4, 발목 peak 168Nm), torqueLimitTask 일반화.
- bridge: 관절 OCS2 jointNames로 동적구성(12/16 자동), 발목홀드 조건부
  (16-DOF는 WBC제어→홀드0), rbd/torque/metric 루프 nJ화, jointVel idx 12+nJ.
- ★GEARBOX(반사관성, A quad_control.hpp:107 이식): dof_armature=I_rot·N²
  +damping+friction(hip7·thigh7·calf10.5·foot8.4). MJCF 0→flail 과장 보정,
  버징에도 도움. 기본ON(GEARBOX=0으로 끔).

검증: 모델로드 OK(mass38·state28·genCoord22·STANCE 힘균형 Fz≈mg).
16-DOF STANCE solid(z0.46·tilt<0.85°·qpFail0·nineq52). 16-DOF TROT 보행
(0.3m/s 추종·base_x 1.96m·6.5s+)·★버징 frontJvPk 26→평균1~6(능동발목+
gearbox 흡수). 단 tilt 간헐스파이크·qpFail 발생=ankle Q/R·토크한계 미튜닝
(12-DOF보다 덜 다듬어짐, 튜닝 후속).

Co-Authored-By: Claude Opus 4.8 <noreply@anthropic.com>

File: quad/ocs2_02leg/urdf/02leg_ocs2_12dof.urdf (robot description, URDF)
Before this commit: robot 02_Leg_UFDF_260703_2, 22 links, 21 joints
Joints:
- joint FL_foot_joint: type revolute -> fixed
- joint FR_foot_joint: type revolute -> fixed
- joint HL_foot_joint: type revolute -> fixed
- joint HR_foot_joint: type revolute -> fixed
